File: PCB/Brain_Rot_Pod_Nano_PCB/Brain_Rot_Pod_Nano_PCB.kicad_sch (KiCad schematic)
At the start: 21 parts, among them J1 USB_C_Receptacle_USB2.0_16P, J2 JST_Battery_Conn, J3 AudioJack3_Switch, J4 ST7789 Display Header, J5 Micro_SD_Card, Q1 FS8205, Q2 AO3400A, SW1 RotaryEncoder_Switch, SW2 UI1, SW3 UI2, SW4 UI3, SW5 UI4, SW6 BOOT, SW7 ABORT, U1 ESP32-S3-WROOM-1, U2 TP4056, U3 DW01A, U4 AP2112K-3.3, U5 PCM5102A, U6 MAX98357A

Commit message: updated journal and other files
Parts:
- added C1, C15, C18, C2, C4, C5, C8: 10uF, symbol Device:C
- added C10, C11, C14, C16, C17, C3, C6, C7, C9: 0.1uF, symbol Device:C
- added C12, C13: 2.2uF, symbol Device:C
- added D1: RLED, symbol Device:LED
- added D2: GLED, symbol Device:LED
- added R1, R2: 5.1kR, symbol Device:R
- added R10, R6, R9: 100R, symbol Device:R
- added R11, R12, R13, R16, R17, R8: 10kR, symbol Device:R
- added R14, R4, R5, R7: 1kR, symbol Device:R
- added R15: 100kR, symbol Device:R
- added R3: 4.7kR, symbol Device:R
- added SW8: EN_PUSH, symbol Switch:SW_Push
- added SW9: SW_Push, symbol Switch:SW_Push
Connections:
- net GND: now reaches SW6.1
- net GND: now also J1.A1 (GND), J1.A12 (GND), J1.B1 (GND), J1.B12 (GND), J1.S1 (SHIELD), J3.S, J4.1 (Pin_1), J5.6 (VSS), J5.9 (SHIELD), Q1.1, Q2.2 (S), SW1.C, SW1.S1, SW2.1, SW3.1, SW4.1, SW5.1, SW7.1, U1.1 (GND), U1.40 (GND), U1.41 (GND), U2.1 (TEMP), U2.3 (GND), U2.9 (EPAD), U4.2 (GND), U5.10 (DEMP), U5.11 (FLT), U5.12 (SCK), U5.16 (FMT), U5.19 (DGND), U5.3 (CPGND), U5.9 (AGND), U6.11 (GND), U6.15 (GND), U6.17 (PAD), U6.2 (GAIN_SLOT), U6.3 (GND), C1.1, C10.1, C11.1, C13.2, C14.2, C15.2, C16.2, C17.1, C18.1, C2.1, C4.2, C5.2, C6.2, C7.2, C8.2, C9.1, R1.1, R15.2, R2.1, R3.2, R7.2, SW8.1, SW9.1
- net IO0: now reaches SW6.2
- net IO0: now also U1.27 (IO0), R17.1, SW9.2
- net at U2.2 (PROG): now also R3.1
- net at U2.4 (V_{CC}): now also J1.A4 (VBUS), J1.A9 (VBUS), J1.B4 (VBUS), J1.B9 (VBUS), U2.8 (CE), C1.2, R4.1, R5.1
- net VBAT: now reaches U2.5 (BAT)
- net VBAT: now also J2.1 (Pin_1), U4.1 (VIN), U4.3 (EN), U6.4 (~{SD_MODE}), U6.7 (VDD), U6.8 (VDD), C2.2, C4.1, C7.1, C8.1, R6.2
- net at U2.6 (~{STDBY}): now also D2.1 (K)
- net at U2.7 (~{CHRG}): now also D1.1 (K)
- net 3V3: now reaches U5.1 (CPVDD)
- net 3V3: now also J4.2 (Pin_2), J5.4 (VDD), U1.2 (3V3), U4.5 (VOUT), U5.20 (DVDD), U5.8 (AVDD), C10.2, C11.2, C15.1, C16.1, C17.2, C18.2, C5.1, C6.1, C9.2, R11.2, R12.2, R13.2, R16.2, R17.2, R8.2
- net I2S_BCLK: now reaches U5.13 (BCK)
- net I2S_BCLK: now also U1.4 (IO4), U6.16 (BCLK)
- net I2S_DOUT: now reaches U5.14 (DIN)
- net I2S_DOUT: now also U1.6 (IO6), U6.1 (DIN)
- net I2S_LRCLK: now reaches U5.15 (LRCK)
- net I2S_LRCLK: now also U1.5 (IO5), U6.14 (LRCLK)
- net at U5.17 (XSMT): now also R8.1
- net at U5.18 (LDOO): now also C14.1
- net at U5.2 (CAPP): now also C12.1
- net at U5.4 (CAPM): now also C12.2
- net at U5.5 (VNEG): now also C13.1
- net at U5.6 (OUTL): now also R9.1
- net at U5.7 (OUTR): now also R10.1
- net UI_RIGHT: now reaches SW5.2
- net UI_RIGHT: now also U1.21 (IO13)
- net at Q2.1 (G): now also R14.2, R15.1
- net at Q2.3 (D): now also J4.8 (Pin_8)
- net UI_DOWN: now reaches SW4.2
- net UI_DOWN: now also U1.19 (IO11)
- net at J1.A5 (CC1): now also R1.2
- net USB_D+: now reaches J1.A6 (D+)
- net USB_D+: now also J1.B6 (D+), U1.14 (USB_D+)
- net USB_D-: now reaches J1.A7 (D-)
- net USB_D-: now also J1.B7 (D-), U1.13 (USB_D-)
- net at J1.B5 (CC2): now also R2.2
- net at LS1.1: now also U6.9 (OUTP)
- net at LS1.2: now also U6.10 (OUTN)
- net GND_BAT: now reaches J2.2 (Pin_2)
- net GND_BAT: now also Q1.3, U3.6 (GND), C3.1
- net ENC_A: now reaches SW1.A
- net ENC_A: now also U1.22 (IO14)
- net ENC_B: now reaches SW1.B
- net ENC_B: now also U1.8 (IO15)
- net ENC_SW: now reaches SW1.S2
- net ENC_SW: now also U1.9 (IO16)
- net ABORT_BTN: now reaches SW7.2
- net ABORT_BTN: now also U1.39 (IO1)
- net UI_LEFT: now reaches SW3.2
- net UI_LEFT: now also U1.20 (IO12)
- net at J3.R: now also R10.2
- net at J3.T: now also R9.2
- net UI_UP: now reaches SW2.2
- net UI_UP: now also U1.18 (IO10)
- net at Q1.4: now also U3.3 (OC)
- net at Q1.6: now also U3.1 (OD)
- net SD_CS: now reaches J5.2 (DAT3/CD)
- net SD_CS: now also U1.35 (IO42), R11.1
- net SPI_MOSI: now reaches J5.3 (CMD)
- net SPI_MOSI: now also J4.4 (Pin_4), U1.28 (IO35), R12.1
- net SPI_SCK: now reaches J5.5 (CLK)
- net SPI_SCK: now also J4.3 (Pin_3), U1.29 (IO36)
- net SPI_MISO: now reaches J5.7 (DAT0)
- net SPI_MISO: now also U1.30 (IO37), R13.1
- net at U3.2 (CS): now also R7.1
- net at U3.5 (VCC): now also C3.2, R6.1
- net EN: now reaches U1.3 (EN)
- net EN: now also R16.1, SW8.2
- net TFT_CS: now reaches U1.31 (IO38)
- net TFT_CS: now also J4.7 (Pin_7)
- net TFT_DC: now reaches U1.32 (IO39)
- net TFT_DC: now also J4.6 (Pin_6)
- net TFT_RST: now reaches U1.33 (IO40)
- net TFT_RST: now also J4.5 (Pin_5)
- net TFT_BLK: now reaches U1.34 (IO41)
- net TFT_BLK: now also R14.1
- new net: D2.2 (A), R5.2
- new net: D1.2 (A), R4.2
- no-connect marks 0 -> 22
Other:
- moved on the sheet: J1, J2, J3, J4, LS1, Q1, Q2, SW1, SW2, SW3, SW4, SW5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

Commit message: finished PCB
Parts:
- removed J4: ST7789 Display Header, symbol Connector:Conn_01x08_Pin
- removed Q2: AO3400A, Package_TO_SOT_SMD:SOT-23, symbol Transistor_FET:AO3400A
- removed R14: 1kR, symbol Device:R
- removed R15: 100kR, symbol Device:R
- added J4: TFT_Conn, Connector_PinHeader_2.54mm:PinHeader_1x09_P2.54mm_Vertical, symbol Connector_Generic:Conn_01x09
- added SW10: UI4, Button_Switch_Keyboard:SW_Cherry_MX_1.00u_PCB, symbol Switch:SW_Push
- C1, C10, C11, C12, C13, C14, C15, C16, C17, C18, C2, C3, C4, C5, C6, C7, C8, C9: footprint (none) -> Capacitor_SMD:C_0805_2012Metric
- D1, D2: footprint (none) -> LED_SMD:LED_0805_2012Metric
- J1: footprint (none) -> Connector_USB:USB_C_Receptacle_HRO_TYPE-C-31-M-12
- J2, LS1: footprint (none) -> Connector_JST:JST_PH_S2B-PH-K_1x02_P2.00mm_Horizontal
- J3: footprint (none) -> Connector_Audio:Jack_3.5mm_CUI_SJ1-3523N_Horizontal
- J5: footprint (none) -> Connector_Card:microSD_HC_Hirose_DM3AT-SF-PEJM5
- Q1: footprint FS8205:SOT95P280X145-6N -> Package_SO:TSSOP-8_4.4x3mm_P0.65mm
- R1, R10, R16, R17, R2, R3, R4, R5, R6, R7, R8, R9: footprint (none) -> Resistor_SMD:R_0805_2012Metric
- R11, R12, R13: value 10kR -> 4.7kR; footprint (none) -> Resistor_SMD:R_0805_2012Metric
- SW1: footprint (none) -> Rotary_Encoder:RotaryEncoder_Alps_EC11E-Switch_Vertical_H20mm
- SW2, SW3, SW4, SW5, SW6, SW7: footprint (none) -> Button_Switch_Keyboard:SW_Cherry_MX_1.00u_PCB
- SW8: footprint (none) -> Button_Switch_THT:SW_PUSH-12mm
- SW9: value SW_Push -> IO0_Push; footprint (none) -> Button_Switch_THT:SW_PUSH-12mm
Connections:
- net 3V3: now also J4.1 (Pin_1), J4.8 (Pin_8)
- net GND: now also J4.2 (Pin_2), SW10.1
- net IO0: now also SW5.2; no longer SW6.2
- net SPI_MISO: now also J4.9 (Pin_9)
- net SPI_MOSI: now also J4.6 (Pin_6)
- net SPI_SCK: now also J4.7 (Pin_7)
- net TFT_CS: now also J4.3 (Pin_3)
- net TFT_DC: now also J4.5 (Pin_5)
- net TFT_RST: now also J4.4 (Pin_4)
- net UI_LEFT: now also SW10.2; no longer SW3.2
- net UI_RIGHT: now also SW2.2; no longer SW5.2
- net UI_UP: now also SW6.2; no longer SW2.2
- net UI_SELECT: now reaches U1.17 (IO9)
- net UI_SELECT: now also SW3.2
- no-connect marks 22 -> 18
Other:
- moved on the sheet: C10, C11, C12, C13, C14, C9, R10, R8, R9, SW1, SW2, SW3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
